File: Hardware/Flight_Board/Microcontroller.kicad_sch (KiCad schematic)
At the start: 20 parts, among them J3 Conn_01x04, J4 Conn_01x06, SW1 SW_Push, U1 FT5HN

Commit message: initial route of 4-layer board
ouch
Parts:
- removed C2: 100n, Capacitor_SMD:C_0603_1608Metric_Pad1.08x0.95mm_HandSolder, symbol Device:C
- removed SW1: SW_Push, Button_Switch_SMD:SW_SPST_PTS645, symbol Switch:SW_Push
- renumbered R1 to R4, R2 to R5, R3 to R6
Other:
- note removed: "Reset Switch"
