File: Hardware/Flight_Board/Barometer.kicad_sch (KiCad schematic)
At the start: 1 part

Commit message: Make Barometer
Parts:
- added C1, C2: 100n, symbol Device:C
Connections:
- net VDDio: now reaches U5.1 (VDDIO)
- net VDDio: now also C1.1
- net VDD: now reaches U5.10 (VDD)
- net VDD: now also C2.1
- net SCK: now reaches U5.2 (SCK)
- net GND: now reaches U5.3 (VSS)
- net GND: now also U5.8 (VSS), U5.9 (VSS), C1.2, C2.2
- net SDI: now reaches U5.4 (SDI)
- net SDO: now reaches U5.5 (SDO)
- net CSB: now reaches U5.6 (CSB)
- net INT: now reaches U5.7 (INT)
Changed lines of the file:
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@@
 (kicad_sch (version 20230121) (generator eeschema)
   (paper "A4")
+  (junction (at 185.42 78.74) (diameter 0) (color 0 0 0 0)
+  )
+  (junction (at 172.72 114.3) (diameter 0) (color 0 0 0 0)
+  )
+  (junction (at 185.42 109.22) (diameter 0) (color 0 0 0 0)
+  )
+  (junction (at 185.42 114.3) (diameter 0) (color 0 0 0 0)
+  )
+  (junction (at 115.57 69.85) (diameter 0) (color 0 0 0 0)
+  )
+  (junction (at 185.42 106.68) (diameter 0) (color 0 0 0 0)
+  )
+  (wire (pts (xy 177.8 106.68) (xy 185.42 106.68))
+    (stroke (width 0) (type default))
+  )
+  (wire (pts (xy 115.57 69.85) (xy 172.72 69.85))
+    (stroke (width 0) (type default))
+  )
+  (wire (pts (xy 130.81 87.63) (xy 162.56 87.63))
+    (stroke (width 0) (type default))
+  )
+  (wire (pts (xy 185.42 78.74) (xy 177.8 78.74))
+    (stroke (width 0) (type default))
+  )
+  (wire (pts (xy 175.26 109.22) (xy 185.42 109.22))
+    (stroke (width 0) (type default))
+  )
+  (wire (pts (xy 115.57 68.58) (xy 115.57 69.85))
+    (stroke (width 0) (type default))
+  )
+  (wire (pts (xy 115.57 99.06) (xy 115.57 114.3))
+    (stroke (width 0) (type default))
+  )
+  (wire (pts (xy 185.42 109.22) (xy 185.42 106.68))
+    (stroke (width 0) (type default))
+  )
+  (wire (pts (xy 185.42 109.22) (xy 185.42 114.3))
+    (stroke (width 0) (type default))
+  )
+  (wire (pts (xy 172.72 69.85) (xy 172.72 78.74))
+    (stroke (width 0) (type default))
+  )
+  (wire (pts (xy 130.81 97.79) (xy 162.56 97.79))
+    (stroke (width 0) (type default))
+  )
+  (wire (pts (xy 115.57 114.3) (xy 172.72 114.3))
+    (stroke (width 0) (type default))
+  )
+  (wire (pts (xy 175.26 106.68) (xy 175.26 109.22))
+    (stroke (width 0) (type default))
+  )
+  (wire (pts (xy 130.81 95.25) (xy 162.56 95.25))
+    (stroke (width 0) (type default))
+  )
+  (wire (pts (xy 185.42 114.3) (xy 172.72 114.3))
+    (stroke (width 0) (type default))
+  )
+  (wire (pts (xy 115.57 69.85) (xy 115.57 91.44))
+    (stroke (width 0) (type default))
+  )
+  (wire (pts (xy 130.81 90.17) (xy 162.56 90.17))
+    (stroke (width 0) (type default))
+  )
+  (wire (pts (xy 172.72 114.3) (xy 172.72 106.68))
+    (stroke (width 0) (type default))
+  )
+  (wire (pts (xy 185.42 106.68) (xy 185.42 96.52))
+    (stroke (width 0) (type default))
+  )
+  (wire (pts (xy 116.84 68.58) (xy 115.57 68.58))
+    (stroke (width 0) (type default))
+  )
+  (wire (pts (xy 185.42 88.9) (xy 185.42 78.74))
+    (stroke (width 0) (type default))
+  )
+  (wire (pts (xy 185.42 71.12) (xy 185.42 78.74))
+    (stroke (width 0) (type default))
+  )
+  (wire (pts (xy 130.81 92.71) (xy 162.56 92.71))
+    (stroke (width 0) (type default))
+  )
+  (wire (pts (xy 185.42 116.84) (xy 185.42 114.3))
+    (stroke (width 0) (type default))
+  )
+  (hierarchical_label "VDD" (shape input) (at 185.42 71.12 0) (fields_autoplaced)
+    (effects (font (size 1.27 1.27)) (justify left))
+  )
+  (hierarchical_label "SCK" (shape input) (at 130.81 87.63 180) (fields_autoplaced)
+    (effects (font (size 1.27 1.27)) (justify right))
+  )
+  (hierarchical_label "SDI" (shape input) (at 130.81 90.17 180) (fields_autoplaced)
+    (effects (font (size 1.27 1.27)) (justify right))
+  )
+  (hierarchical_label "CSB" (shape input) (at 130.81 95.25 180) (fields_autoplaced)
+    (effects (font (size 1.27 1.27)) (justify right))
+  )
+  (hierarchical_label "VDDio" (shape input) (at 116.84 68.58 0) (fields_autoplaced)
+    (effects (font (size 1.27 1.27)) (justify left))
+  )
+  (hierarchical_label "INT" (shape input) (at 130.81 97.79 180) (fields_autoplaced)
+    (effects (font (size 1.27 1.27)) (justify right))
+  )
+  (hierarchical_label "SDO" (shape input) (at 130.81 92.71 180) (fields_autoplaced)
+    (effects (font (size 1.27 1.27)) (justify right))
+  )
+  (symbol (lib_id "Device:C") (at 115.57 95.25 0) (unit 1)
+    (in_bom yes) (on_board yes) (dnp no) (fields_autoplaced)
+    (property "Reference" "C1" (at 119.38 93.98 0)
+      (effects (font (size 1.27 1.27)) (justify left))
+    )
+    (property "Value" "100n" (at 119.38 96.52 0)
+      (effects (font (size 1.27 1.27)) (justify left))
+    )
+    (property "Footprint" "" (at 116.5352 99.06 0)
+      (effects (font (size 1.27 1.27)) hide)
+    )
+    (property "Datasheet" "~" (at 115.57 95.25 0)
+      (effects (font (size 1.27 1.27)) hide)
+    )
+    (pin "1")
+    (pin "2")
+    (instances
+      (project "Flight_Board"
+        (path "/e8eb85d5-f1ff-4500-895d-25b9ff5f6d36/438715e3-b069-4320-9581-dc19d9c2cf0e"
+          (reference "C1") (unit 1)
+        )
+      )
+    )
+  )
+  (symbol (lib_id "Device:C") (at 185.42 92.71 0) (unit 1)
+    (in_bom yes) (on_board yes) (dnp no) (fields_autoplaced)
+    (property "Reference" "C2" (at 189.23 91.44 0)
+      (effects (font (size 1.27 1.27)) (justify left))
+    )
+    (property "Value" "100n" (at 189.23 93.98 0)
+      (effects (font (size 1.27 1.27)) (justify left))
+    )
+    (property "Footprint" "" (at 186.3852 96.52 0)
+      (effects (font (size 1.27 1.27)) hide)
+    )
+    (property "Datasheet" "~" (at 185.42 92.71 0)
+      (effects (font (size 1.27 1.27)) hide)
+    )
+    (pin "1")
+    (pin "2")
+    (instances
+      (project "Flight_Board"
+        (path "/e8eb85d5-f1ff-4500-895d-25b9ff5f6d36/438715e3-b069-4320-9581-dc19d9c2cf0e"
+          (reference "C2") (unit 1)
+        )
+      )
+    )
+  )
   (symbol (lib_id "Project:BMP390") (at 175.26 92.71 0) (unit 1)
     (in_bom yes) (on_board yes) (dnp no) (fields_autoplaced)
@@
         )
       )
+    )
+  )
+  (symbol (lib_id "power:GND") (at 185.42 116.84 0) (unit 1)
+    (in_bom yes) (on_board yes) (dnp no) (fields_autoplaced)
+    (property "Reference" "#PWR016" (at 185.42 123.19 0)
+      (effects (font (size 1.27 1.27)) hide)
+    )
+    (property "Value" "GND" (at 185.42 121.92 0)
+      (effects (font (size 1.27 1.27)))
+    )
+    (property "Footprint" "" (at 185.42 116.84 0)
+      (effects (font (size 1.27 1.27)) hide)
+    )
+    (property "Datasheet" "" (at 185.42 116.84 0)
+      (effects (font (size 1.27 1.27)) hide)
+    )
+    (pin "1")
+    (instances
+      (project "Flight_Board"
+        (path "/e8eb85d5-f1ff-4500-895d-25b9ff5f6d36/438715e3-b069-4320-9581-dc19d9c2cf0e"
+          (reference "#PWR016") (unit 1)
+        )
+      )
