File: Hardware/Flight_Board/LoRa.kicad_sch (KiCad schematic)
At the start: 1 part

Commit message: Updated Lora Board
Connections:
- net RADIO_BUSY renamed LORA_BUSY
- removed net RADIO_DIO1: U8.4 (DIO1), U8.6 (SCK), U8.7 (MOSI), U8.8 (MISO)
- new net LORA_DIO1: U8.4 (DIO1)
- new net LORA_SCK: U8.6 (SCK)
- new net LORA_SDI: U8.7 (MOSI)
- new net LORA_SDO: U8.8 (MISO)
Changed lines of the file:
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@@
     (stroke (width 0) (type default))
   )
-  (hierarchical_label "RADIO_DIO1" (shape bidirectional) (at 144.78 86.36 0) (fields_autoplaced)
+  (hierarchical_label "LORA_SDI" (shape input) (at 144.78 88.9 0) (fields_autoplaced)
     (effects (font (size 1.27 1.27)) (justify left))
   )
@@
     (effects (font (size 1.27 1.27)) (justify left))
   )
-  (hierarchical_label "RADIO_DIO1" (shape bidirectional) (at 116.84 93.98 180) (fields_autoplaced)
+  (hierarchical_label "LORA_DIO1" (shape bidirectional) (at 116.84 93.98 180) (fields_autoplaced)
     (effects (font (size 1.27 1.27)) (justify right))
   )
-  (hierarchical_label "RADIO_DIO1" (shape bidirectional) (at 144.78 88.9 0) (fields_autoplaced)
+  (hierarchical_label "LORA_SCK" (shape bidirectional) (at 144.78 86.36 0) (fields_autoplaced)
     (effects (font (size 1.27 1.27)) (justify left))
   )
-  (hierarchical_label "RADIO_BUSY" (shape bidirectional) (at 116.84 91.44 180) (fields_autoplaced)
+  (hierarchical_label "LORA_BUSY" (shape bidirectional) (at 116.84 91.44 180) (fields_autoplaced)
     (effects (font (size 1.27 1.27)) (justify right))
   )
-  (hierarchical_label "RADIO_DIO1" (shape bidirectional) (at 144.78 91.44 0) (fields_autoplaced)
+  (hierarchical_label "LORA_SDO" (shape output) (at 144.78 91.44 0) (fields_autoplaced)
     (effects (font (size 1.27 1.27)) (justify left))
   )
