File: Hardware/Flight_Board/Flight_Board.kicad_sch (KiCad schematic)
At the start: 0 parts

Commit message: Updated Lora Board
Other:
- sheet LoRa ports: added LORA_BUSY, LORA_DIO1, LORA_NSS, LORA_SCK, LORA_SDI, LORA_SDO; removed none
Changed lines of the file:
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@@
+    (stroke (width 0) (type default))
+  )
+  (wire (pts (xy 129.54 40.64) (xy 139.7 40.64))
     (stroke (width 0) (type default))
   )
@@
     (stroke (width 0) (type default))
   )
+  (wire (pts (xy 129.54 43.18) (xy 139.7 43.18))
+    (stroke (width 0) (type default))
+  )
+  (wire (pts (xy 129.54 48.26) (xy 139.7 48.26))
+    (stroke (width 0) (type default))
+  )
   (wire (pts (xy 238.76 43.18) (xy 233.68 43.18))
     (stroke (width 0) (type default))
@@
     (stroke (width 0) (type default))
   )
+  (wire (pts (xy 129.54 50.8) (xy 139.7 50.8))
+    (stroke (width 0) (type default))
+  )
+  (wire (pts (xy 129.54 45.72) (xy 139.7 45.72))
+    (stroke (width 0) (type default))
+  )
   (wire (pts (xy 127 63.5) (xy 139.7 63.5))
     (stroke (width 0) (type default))
@@
   )
   (wire (pts (xy 233.68 43.18) (xy 233.68 68.58))
+    (stroke (width 0) (type default))
+  )
+  (wire (pts (xy 129.54 38.1) (xy 139.7 38.1))
     (stroke (width 0) (type default))
   )
@@
       (effects (font (size 1.27 1.27)) (justify left top))
     )
-    (instances
+    (pin "LORA_NSS" bidirectional (at 129.54 45.72 0)
+      (effects (font (size 1.27 1.27)) (justify right))
+    )
+    (pin "LORA_SCK" bidirectional (at 129.54 43.18 0)
+      (effects (font (size 1.27 1.27)) (justify right))
+    )
+    (pin "LORA_SDI" input (at 129.54 40.64 0)
+      (effects (font (size 1.27 1.27)) (justify right))
+    )
+    (pin "LORA_SDO" output (at 129.54 38.1 0)
+      (effects (font (size 1.27 1.27)) (justify right))
+    )
+    (pin "LORA_BUSY" bidirectional (at 129.54 48.26 0)
+      (effects (font (size 1.27 1.27)) (justify right))
+    )
+    (pin "LORA_DIO1" bidirectional (at 129.54 50.8 0)
+      (effects (font (size 1.27 1.27)) (justify right))
+    )
+    (instances

Commit message: clean up and finalize initial design
Parts:
- added J1: Conn_01x04, symbol Connector_Generic:Conn_01x04
- added J2: Conn_01x08, symbol Connector_Generic:Conn_01x08
Connections:
- new net GND: J1.2 (Pin_2), J1.4 (Pin_4), J2.2 (Pin_2), J2.4 (Pin_4), J2.6 (Pin_6), J2.8 (Pin_8)
- new net PYRO1: J2.1 (Pin_1)
- new net PYRO2: J2.3 (Pin_3)
- new net PYRO3: J2.5 (Pin_5)
- new net PYRO4: J2.7 (Pin_7)
- new net VBAT: J1.1 (Pin_1)
- new net VPYRO: J1.3 (Pin_3)
Other:
- sheet Current Switch ports: added EN4, OUT4, VPYRO, ~{ST4}; removed CL, DIAG_EN, VDD_currentswitch
- sheet LoRa ports: added LORA_RST; removed none
- sheet Microcontroller ports: added RADIO_RST, SW_EN1, SW_EN2, SW_EN3, SW_EN4, SW_ST1, SW_ST2, SW_ST3, SW_ST4, VBAT; removed VBAT_ADC
- sheet Power ports: added Vin, Vout; removed none
- note removed: "LR62 Radio goes here"
- note removed: "Set INPUT_PULLUP in software to cover ~{ST1,2,3} pullups"
- note removed: "TPS current limiter goes here"

Commit message: clean up, implement suggestions from saunders
Parts:
- added R31, R33, R34: 22k, symbol Device:R
Connections:
- net +3.3V: now also R31.1, R33.1, R34.1
- net Barometer/SDO: now also R31.2
- net Barometer/~{CS}: now also R33.2
- net IMU/~{CS}: now also R34.2
Other:
- sheet Accelerometer ports: added none; removed INT2
- sheet GPS ports: added none; removed SCL, SDA, TIMEPULSE
- sheet IMU ports: added none; removed INT2
- sheet Microcontroller ports: added ACCEL_INT, BARO_INT, IMU_INT; removed none
