File: Hardware/Flight_Board/current_switch.kicad_sch (KiCad schematic)
At the start: 29 parts, among them U8 TPS274160A

Commit message: initial route of 4-layer board
ouch
Parts:
- removed D1: P1, LED_SMD:LED_0603_1608Metric_Pad1.05x0.95mm_HandSolder, symbol Device:LED
- removed D1: P4, LED_SMD:LED_0603_1608Metric_Pad1.05x0.95mm_HandSolder, symbol Device:LED
- removed D1: P2, LED_SMD:LED_0603_1608Metric_Pad1.05x0.95mm_HandSolder, symbol Device:LED
- removed D1: P3, LED_SMD:LED_0603_1608Metric_Pad1.05x0.95mm_HandSolder, symbol Device:LED
- removed R26 (x4): 22k, Resistor_SMD:R_0603_1608Metric_Pad0.98x0.95mm_HandSolder, symbol Device:R
- removed R27, R28, R29, R30: 10k, Resistor_SMD:R_0603_1608Metric_Pad0.98x0.95mm_HandSolder, symbol Device:R
- U8: footprint Package_DFN_QFN:QFN-28-1EP_4x5mm_P0.5mm_EP2.65x3.65mm_ThermalVias -> Project:TPS274160A
- renumbered C33 to C31, C34 to C32, C35 to C33, C36 to C34, C37 to C35, C38 to C36, R15 to R18, R16 to R19, R17 to R20, R18 to R21, R19 to R22, R20 to R23, R21 to R24, R22 to R25, R23 to R26, R24 to R27
Other:
- moved on the sheet: C31, C32, C33, C34, C35, C36, R18, R19, R20, R21, R22, R23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
