File: Hardware/Flight_Board/Power.kicad_sch (KiCad schematic)
At the start: 3 parts

Commit message: initial route of 4-layer board
ouch
Parts:
- removed TP1: 3V3, TestPoint:TestPoint_THTPad_2.0x2.0mm_Drill1.0mm, symbol Connector:TestPoint
- added C21: 1u, Capacitor_SMD:C_0603_1608Metric_Pad1.08x0.95mm_HandSolder, symbol Device:C
- added C22: 2.2u, Capacitor_SMD:C_0603_1608Metric_Pad1.08x0.95mm_HandSolder, symbol Device:C
- added U7: AP2205-33Y-13, Package_TO_SOT_SMD:SOT-89-3, symbol Project:AP2205-33Y-13
Connections:
- net GND: now also C21.2, C22.2, U7.2 (GND)
- net VBat: now also C21.1, U7.1 (VIN)
- net Vout: now also C22.1, U7.3 (VOUT)
Changed lines of the file:
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@@
 (kicad_sch (version 20230121) (generator eeschema)
   (paper "A4")
+  (junction (at 125.73 82.55) (diameter 0) (color 0 0 0 0)
+  )
+  (junction (at 107.95 92.71) (diameter 0) (color 0 0 0 0)
+  )
+  (junction (at 90.17 82.55) (diameter 0) (color 0 0 0 0)
+  )
   (junction (at 140.97 82.55) (diameter 0) (color 0 0 0 0)
   )
-  (wire (pts (xy 106.68 97.79) (xy 106.68 100.33))
+  (wire (pts (xy 115.57 82.55) (xy 125.73 82.55))
+    (stroke (width 0) (type default))
+  )
+  (wire (pts (xy 125.73 92.71) (xy 125.73 90.17))
+    (stroke (width 0) (type default))
+  )
+  (wire (pts (xy 90.17 92.71) (xy 107.95 92.71))
+    (stroke (width 0) (type default))
+  )
+  (wire (pts (xy 90.17 82.55) (xy 100.33 82.55))
+    (stroke (width 0) (type default))
+  )
+  (wire (pts (xy 107.95 90.17) (xy 107.95 92.71))
+    (stroke (width 0) (type default))
+  )
+  (wire (pts (xy 90.17 82.55) (xy 81.28 82.55))
+    (stroke (width 0) (type default))
+  )
+  (wire (pts (xy 125.73 82.55) (xy 140.97 82.55))
+    (stroke (width 0) (type default))
+  )
+  (wire (pts (xy 107.95 92.71) (xy 107.95 95.25))
     (stroke (width 0) (type default))
   )
@@
     (stroke (width 0) (type default))
   )
+  (wire (pts (xy 107.95 92.71) (xy 125.73 92.71))
+    (stroke (width 0) (type default))
+  )
   (wire (pts (xy 140.97 82.55) (xy 153.67 82.55))
+    (stroke (width 0) (type default))
+  )
+  (wire (pts (xy 90.17 90.17) (xy 90.17 92.71))
     (stroke (width 0) (type default))
   )
@@
     (effects (font (size 1.27 1.27)) (justify left))
   )
-  (hierarchical_label "VBat" (shape input) (at 101.6 82.55 180) (fields_autoplaced)
+  (hierarchical_label "VBat" (shape input) (at 81.28 82.55 180) (fields_autoplaced)
     (effects (font (size 1.27 1.27)) (justify right))
   )
@@
         )
         (path "/e8eb85d5-f1ff-4500-895d-25b9ff5f6d36/bc23ea56-d50e-4ce7-856f-e38dfbe72971"
-          (reference "#PWR073") (unit 1)
+          (reference "#PWR049") (unit 1)
+        )
+      )
+    )
+  )
+  (symbol (lib_id "Device:C") (at 125.73 86.36 0) (unit 1)
+    (in_bom yes) (on_board yes) (dnp no) (fields_autoplaced)
+    (property "Reference" "C22" (at 129.54 85.09 0)
+      (effects (font (size 1.27 1.27)) (justify left))
+    )
+    (property "Value" "2.2u" (at 129.54 87.63 0)
+      (effects (font (size 1.27 1.27)) (justify left))
+    )
+    (property "Footprint" "Capacitor_SMD:C_0603_1608Metric_Pad1.08x0.95mm_HandSolder" (at 126.6952 90.17 0)
+      (effects (font (size 1.27 1.27)) hide)
+    )
+    (property "Datasheet" "~" (at 125.73 86.36 0)
+      (effects (font (size 1.27 1.27)) hide)
+    )
+    (pin "1")
+    (pin "2")
+    (instances
+      (project "Flight_Board"
+        (path "/e8eb85d5-f1ff-4500-895d-25b9ff5f6d36/bc23ea56-d50e-4ce7-856f-e38dfbe72971"
+          (reference "C22") (unit 1)
+        )
+      )
+    )
+  )
+  (symbol (lib_id "Project:AP2205-33Y-13") (at 107.95 82.55 0) (unit 1)
+    (in_bom yes) (on_board yes) (dnp no) (fields_autoplaced)
+    (property "Reference" "U7" (at 107.95 76.2 0)
+      (effects (font (size 1.27 1.27)))
+    )
+    (property "Value" "AP2205-33Y-13" (at 107.95 78.74 0)
+      (effects (font (size 1.27 1.27)))
+    )
+    (property "Footprint" "Package_TO_SOT_SMD:SOT-89-3" (at 107.95 76.835 0)
+      (effects (font (size 1.27 1.27)) hide)
+    )
+    (property "Datasheet" "https://www.diodes.com/assets/Datasheets/AP2205.pdf" (at 107.95 82.55 0)
+      (effects (font (size 1.27 1.27)) hide)
+    )
+    (pin "1")
+    (pin "2")
+    (pin "3")
+    (instances
+      (project "Flight_Board"
+        (path "/e8eb85d5-f1ff-4500-895d-25b9ff5f6d36/bc23ea56-d50e-4ce7-856f-e38dfbe72971"
+          (reference "U7") (unit 1)
+        )
+      )
+    )
+  )
+  (symbol (lib_id "Device:C") (at 90.17 86.36 0) (unit 1)
+    (in_bom yes) (on_board yes) (dnp no) (fields_autoplaced)
+    (property "Reference" "C21" (at 93.98 85.09 0)
+      (effects (font (size 1.27 1.27)) (justify left))
+    )
+    (property "Value" "1u" (at 93.98 87.63 0)
+      (effects (font (size 1.27 1.27)) (justify left))
+    )
+    (property "Footprint" "Capacitor_SMD:C_0603_1608Metric_Pad1.08x0.95mm_HandSolder" (at 91.1352 90.17 0)
+      (effects (font (size 1.27 1.27)) hide)
+    )
+    (property "Datasheet" "~" (at 90.17 86.36 0)
+      (effects (font (size 1.27 1.27)) hide)
+    )
+    (pin "1")
+    (pin "2")
+    (instances
+      (project "Flight_Board"
+        (path "/e8eb85d5-f1ff-4500-895d-25b9ff5f6d36/bc23ea56-d50e-4ce7-856f-e38dfbe72971"
+          (reference "C21") (unit 1)
         )
       )
@@
         )
         (path "/e8eb85d5-f1ff-4500-895d-25b9ff5f6d36/bc23ea56-d50e-4ce7-856f-e38dfbe72971"
-          (reference "D3") (unit 1)
-        )
-      )
-    )
-  )
-  (symbol (lib_id "Connector:TestPoint") (at 140.97 82.55 0) (unit 1)
-    (in_bom yes) (on_board yes) (dnp no)
-    (property "Reference" "TP1" (at 139.7 77.47 90)
-      (effects (font (size 1.27 1.27)) (justify left) hide)
-    )
-    (property "Value" "3V3" (at 142.24 78.74 0)
-      (effects (font (size 1.27 1.27)) (justify left))
-    )
-    (property "Footprint" "TestPoint:TestPoint_THTPad_2.0x2.0mm_Drill1.0mm" (at 146.05 82.55 0)
-      (effects (font (size 1.27 1.27)) hide)
-    )
-    (property "Datasheet" "~" (at 146.05 82.55 0)
-      (effects (font (size 1.27 1.27)) hide)
-    )
-    (pin "1")
-    (instances
-      (project "Flight_Board"
-        (path "/e8eb85d5-f1ff-4500-895d-25b9ff5f6d36/52cae81a-54fe-42c0-9a19-be88b271d004"
-          (reference "TP1") (unit 1)
-        )
-        (path "/e8eb85d5-f1ff-4500-895d-25b9ff5f6d36"
-          (reference "TP21") (unit 1)
-        )
-        (path "/e8eb85d5-f1ff-4500-895d-25b9ff5f6d36/bc23ea56-d50e-4ce7-856f-e38dfbe72971"
-          (reference "TP22") (unit 1)
+          (reference "D2") (unit 1)
         )
       )
@@
         )
         (path "/e8eb85d5-f1ff-4500-895d-25b9ff5f6d36/bc23ea56-d50e-4ce7-856f-e38dfbe72971"
-          (reference "R36") (unit 1)
-        )
-      )
-    )
-  )
-  (symbol (lib_id "power:GND") (at 106.68 100.33 0) (unit 1)
+          (reference "R12") (unit 1)
+        )
+      )
+    )
+  )
+  (symbol (lib_id "power:GND") (at 107.95 95.25 0) (unit 1)
     (in_bom yes) (on_board yes) (dnp no)
-    (property "Reference" "#PWR?" (at 106.68 106.68 0)
-      (effects (font (size 1.27 1.27)) hide)
-    )
-    (property "Value" "GND" (at 106.68 104.14 0)
-      (effects (font (size 1.27 1.27)))
-    )
-    (property "Footprint" "" (at 106.68 100.33 0)
-      (effects (font (size 1.27 1.27)) hide)
-    )
-    (property "Datasheet" "" (at 106.68 100.33 0)
+    (property "Reference" "#PWR?" (at 107.95 101.6 0)
+      (effects (font (size 1.27 1.27)) hide)
+    )
+    (property "Value" "GND" (at 107.95 99.06 0)
+      (effects (font (size 1.27 1.27)))
+    )
+    (property "Footprint" "" (at 107.95 95.25 0)
+      (effects (font (size 1.27 1.27)) hide)
+    )
+    (property "Datasheet" "" (at 107.95 95.25 0)
       (effects (font (size 1.27 1.27)) hide)
     )
@@
         )
         (path "/e8eb85d5-f1ff-4500-895d-25b9ff5f6d36/bc23ea56-d50e-4ce7-856f-e38dfbe72971"
-          (reference "#PWR040") (unit 1)
-        )
-      )
+          (reference "#PWR048") (unit 1)
+        )
+      )
