File: Hardware/Flight_Board/Accelerometer.kicad_sch (KiCad schematic)
At the start: 9 parts, among them U3 ADXL375

Commit message: silkscreen cleanup
Parts:
- C12, C13: value 0.1u -> 100n
Changed lines of the file:
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@@
       (effects (font (size 1.27 1.27)) (justify right))
     )
-    (property "Value" "0.1u" (at 165.1 60.96 0)
+    (property "Value" "100n" (at 165.1 60.96 0)
       (effects (font (size 1.27 1.27)) (justify right))
     )
@@
       (effects (font (size 1.27 1.27)) (justify left))
     )
-    (property "Value" "0.1u" (at 195.58 60.96 0)
-      (effects (font (size 1.27 1.27)) (justify left))
-    )
+    (property "Value" "100n" (at 195.58 60.96 0)
+      (effects (font (size 1.27 1.27)) (justify left))
+    )

Commit message: minor tweaks and prettification
Parts:
- TP2: footprint TestPoint:TestPoint_THTPad_2.0x2.0mm_Drill1.0mm -> TestPoint:TestPoint_Pad_D1.0mm
Changed lines of the file:
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@@
       (effects (font (size 1.27 1.27)) (justify left))
     )
-    (property "Footprint" "TestPoint:TestPoint_THTPad_2.0x2.0mm_Drill1.0mm" (at 133.35 73.66 0)
+    (property "Footprint" "TestPoint:TestPoint_Pad_D1.0mm" (at 133.35 73.66 0)
       (effects (font (size 1.27 1.27)) hide)
     )
@@
       (effects (font (size 1.27 1.27)) (justify left))
     )
-    (property "Footprint" "TestPoint:TestPoint_THTPad_2.0x2.0mm_Drill1.0mm" (at 128.27 73.66 0)
+    (property "Footprint" "TestPoint:TestPoint_Pad_D1.0mm" (at 128.27 73.66 0)
       (effects (font (size 1.27 1.27)) hide)
     )
@@
       (effects (font (size 1.27 1.27)) (justify left))
     )
-    (property "Footprint" "TestPoint:TestPoint_THTPad_2.0x2.0mm_Drill1.0mm" (at 123.19 73.66 0)
+    (property "Footprint" "TestPoint:TestPoint_Pad_D1.0mm" (at 123.19 73.66 0)
       (effects (font (size 1.27 1.27)) hide)
     )
