File: Hardware/Flight_Board/IMU.kicad_sch (KiCad schematic)
At the start: 4 parts, among them U6 BMI323

Commit message: minor tweaks and prettification
Parts:
- TP2: footprint TestPoint:TestPoint_THTPad_2.0x2.0mm_Drill1.0mm -> TestPoint:TestPoint_Pad_D1.0mm
Changed lines of the file:
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@@
       (effects (font (size 1.27 1.27)) (justify left))
     )
-    (property "Footprint" "TestPoint:TestPoint_THTPad_2.0x2.0mm_Drill1.0mm" (at 149.86 77.47 0)
+    (property "Footprint" "TestPoint:TestPoint_Pad_D1.0mm" (at 149.86 77.47 0)
       (effects (font (size 1.27 1.27)) hide)
     )
