File: Hardware/Flight_Board/MicroSD.kicad_sch (KiCad schematic)
At the start: 17 parts, among them J5 MEM2067-02-180-00-A_REVB

Commit message: minor tweaks and prettification
Parts:
- TP2: footprint TestPoint:TestPoint_THTPad_2.0x2.0mm_Drill1.0mm -> TestPoint:TestPoint_Pad_D1.0mm
Changed lines of the file:
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@@
       (effects (font (size 1.27 1.27)) (justify left))
     )
-    (property "Footprint" "TestPoint:TestPoint_THTPad_2.0x2.0mm_Drill1.0mm" (at 191.77 104.14 0)
+    (property "Footprint" "TestPoint:TestPoint_Pad_D1.0mm" (at 191.77 104.14 0)
       (effects (font (size 1.27 1.27)) hide)
     )
@@
       (effects (font (size 1.27 1.27)) (justify left))
     )
-    (property "Footprint" "TestPoint:TestPoint_THTPad_2.0x2.0mm_Drill1.0mm" (at 163.83 104.14 0)
+    (property "Footprint" "TestPoint:TestPoint_Pad_D1.0mm" (at 163.83 104.14 0)
       (effects (font (size 1.27 1.27)) hide)
     )
@@
       (effects (font (size 1.27 1.27)) (justify left))
     )
-    (property "Footprint" "TestPoint:TestPoint_THTPad_2.0x2.0mm_Drill1.0mm" (at 182.88 104.14 0)
-      (effects (font (size 1.27 1.27)) hide)
-    )
+    (property "Footprint" "TestPoint:TestPoint_Pad_D1.0mm" (at 182.88 104.14 0)
+      (effects (font (size 1.27 1.27)) hide)
+    )
