File: Hardware/Nucleo_Backpack/Barometer.kicad_sch (KiCad schematic)
At the start: 4 parts, among them U4 BMP390

Commit message: all components now on the backpack
Parts:
- renumbered TP2 to TP3
Changed lines of the file:
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@@
   (symbol (lib_id "Connector:TestPoint") (at 139.7 93.98 0) (unit 1)
     (in_bom yes) (on_board yes) (dnp no)
-    (property "Reference" "TP2" (at 144.78 90.678 90)
+    (property "Reference" "TP3" (at 144.78 90.678 90)
       (effects (font (size 1.27 1.27)) hide)
     )
