File: Hardware/Nucleo_Backpack/IMU.kicad_sch (KiCad schematic)
At the start: 4 parts, among them U6 BMI323

Commit message: all components now on the backpack
Parts:
- renumbered TP2 to TP3
Changed lines of the file:
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@@
   (symbol (lib_id "Connector:TestPoint") (at 144.78 77.47 0) (unit 1)
     (in_bom yes) (on_board yes) (dnp no)
-    (property "Reference" "TP2" (at 149.86 74.168 90)
+    (property "Reference" "TP3" (at 149.86 74.168 90)
       (effects (font (size 1.27 1.27)) hide)
     )
