File: Hardware/Nucleo_Backpack/MicroSD.kicad_sch (KiCad schematic)
At the start: 17 parts, among them J5 MEM2067-02-180-00-A_REVB

Commit message: all components now on the backpack
Parts:
- renumbered TP2 to TP3
Changed lines of the file:
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@@
   (symbol (lib_id "Connector:TestPoint") (at 186.69 104.14 0) (unit 1)
     (in_bom yes) (on_board yes) (dnp no)
-    (property "Reference" "TP2" (at 191.77 100.838 90)
+    (property "Reference" "TP3" (at 191.77 100.838 90)
       (effects (font (size 1.27 1.27)) hide)
     )
@@
   (symbol (lib_id "Connector:TestPoint") (at 168.91 104.14 0) (mirror y) (unit 1)
     (in_bom yes) (on_board yes) (dnp no)
-    (property "Reference" "TP2" (at 163.83 100.838 90)
+    (property "Reference" "TP3" (at 163.83 100.838 90)
       (effects (font (size 1.27 1.27)) hide)
     )
@@
   (symbol (lib_id "Connector:TestPoint") (at 177.8 104.14 0) (unit 1)
     (in_bom yes) (on_board yes) (dnp no)
-    (property "Reference" "TP2" (at 182.88 100.838 90)
-      (effects (font (size 1.27 1.27)) hide)
-    )
+    (property "Reference" "TP3" (at 182.88 100.838 90)
+      (effects (font (size 1.27 1.27)) hide)
+    )
