File: Hardware/Nucleo_Backpack/Accelerometer.kicad_sch (KiCad schematic)
At the start: 9 parts, among them U3 ADXL375

Commit message: all components now on the backpack
Parts:
- renumbered TP2 to TP10, TP2 to TP11, TP2 to TP12
Changed lines of the file:
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@@
   (symbol (lib_id "Connector:TestPoint") (at 128.27 73.66 0) (unit 1)
     (in_bom yes) (on_board yes) (dnp no)
-    (property "Reference" "TP2" (at 133.35 70.358 90)
+    (property "Reference" "TP12" (at 133.35 70.358 90)
       (effects (font (size 1.27 1.27)) hide)
     )
@@
   (symbol (lib_id "Connector:TestPoint") (at 123.19 73.66 0) (unit 1)
     (in_bom yes) (on_board yes) (dnp no)
-    (property "Reference" "TP2" (at 128.27 70.358 90)
+    (property "Reference" "TP11" (at 128.27 70.358 90)
       (effects (font (size 1.27 1.27)) hide)
     )
@@
   (symbol (lib_id "Connector:TestPoint") (at 118.11 73.66 0) (unit 1)
     (in_bom yes) (on_board yes) (dnp no)
-    (property "Reference" "TP2" (at 123.19 70.358 90)
+    (property "Reference" "TP10" (at 123.19 70.358 90)
       (effects (font (size 1.27 1.27)) hide)
     )

Commit message: Backpack Update
Connections:
- no-connect marks 0 -> 1
Changed lines of the file:
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@@
   (junction (at 176.53 92.71) (diameter 0) (color 0 0 0 0)
   )
+  (no_connect (at 160.02 87.63))
   (wire (pts (xy 128.27 85.09) (xy 160.02 85.09))
     (stroke (width 0) (type default))
