File: Hardware/Nucleo_Backpack/Nucleo_Backpack.kicad_pcb (KiCad board)
At the start: 2 copper layers, 70.1 x 57.5 mm, 59 parts, among them J1 CN7, J2 CN10, J4 Conn_01x04, J5 MEM2067-02-180-00-A_REVB, U3 ADXL375, U4 BMP390, U5 FGPMMOPA6H, U6 BMI323, U9 LR62E

Commit message: Backpack Updates
Routing:
- net GND: track 0.00 -> 53.4 mm, vias 0 -> 3
- net SPI1_NSS: track 29.7 -> 71.6 mm, vias 1 -> 3
- net +3.3V: track 219.4 -> 220.1 mm
- added copper zone on B.Cu, net GND
- added copper zone on F.Cu, net GND
Other:
- board size 70.1 x 57.5 mm -> 70 x 57.5 mm

Commit message: Backpack Update
Parts:
- removed C17: 1u, Capacitor_SMD:C_0603_1608Metric_Pad1.08x0.95mm_HandSolder
- removed C18: 100n, Capacitor_SMD:C_0603_1608Metric_Pad1.08x0.95mm_HandSolder
- removed D1: GPS_TX, LED_SMD:LED_0603_1608Metric_Pad1.05x0.95mm_HandSolder
- removed FB2: FerriteBead, Resistor_SMD:R_0603_1608Metric_Pad0.98x0.95mm_HandSolder
- removed H1, H2, H3: MountingHole, MountingHole:MountingHole_3.2mm_M3
- removed R10, R9: 220, Resistor_SMD:R_0603_1608Metric_Pad0.98x0.95mm_HandSolder
- removed R11: 22k, Resistor_SMD:R_0603_1608Metric_Pad0.98x0.95mm_HandSolder
- removed U5: FGPMMOPA6H, Project:FGPMMOPA6H
- moved R1 15.5 mm to (139.3, 91.6)
- moved J4 12.1 mm to (130.5, 107.8)
- moved R2 10.6 mm to (140.8, 91.7), turned to 90 degrees
- moved TP12 6.79 mm to (163.1, 102.2)
- moved TP14 3.06 mm to (163.3, 86.5)
- moved TP13 2.79 mm to (163.4, 89.7)
- moved C15 2.43 mm to (144.9, 86.9)
- moved C16 2.43 mm to (144.9, 88.4)
- moved U4 1.99 mm to (141.0, 87.7)
- moved C12 0.99 mm to (155.1, 62.9)
- moved C28 0.59 mm to (135.5, 66.0)
- moved R16 0.59 mm to (135.5, 64.4)
- moved R7 0.38 mm to (158.1, 65.4)
- moved R17 0.09 mm to (131.4, 64.4)
Connections:
- J2 pad 21: USART1_TX -> unconnected-(J2-Pin_21-Pad21)
- J2 pad 33: USART1_RX -> unconnected-(J2-Pin_33-Pad33)
Routing:
- net USART1_RX: track 65.4 -> 0.00 mm
- net USART1_TX: track 59.4 -> 0.00 mm, vias 2 -> 0
- net +3.3V: track 220.1 -> 177.3 mm, vias 21 -> 16
- net RADIO_DIO1: track 70.0 -> 58.7 mm, vias 0 -> 3
- net USART2_RX: track 26.2 -> 36.4 mm
- net USART2_TX: track 26.6 -> 36.0 mm
- net SPI1_NSS: track 71.6 -> 63.4 mm
- net ACCEL_INT: track 51.0 -> 43.2 mm, vias 1 -> 2
- net SDIO_CMD: track 36.2 -> 29.0 mm, vias 0 -> 2
- net Net-(U5-VCC): track 6.55 -> 0.00 mm
- net SPI2_MISO: track 83.5 -> 88.8 mm, vias 3 -> 2
- net Net-(U5-TX): track 4.89 -> 0.00 mm
- net SDIO_D1: track 43.9 -> 47.4 mm, vias 0 -> 2
- net Net-(U5-RX): track 3.15 -> 0.00 mm
- net SPI2_CS1: track 31.0 -> 33.8 mm, vias 0 -> 2
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
Commit message: cleaned up boards
Routing:
- net +3.3V: track 177.3 -> 182.2 mm
- net GND: track 53.9 -> 56.0 mm, vias 16 -> 58

Commit message: regenerate gerbers
Routing:
- net +3.3V: track 182.2 -> 177.3 mm
- net GND: track 56.0 -> 53.9 mm, vias 58 -> 16
